Commit message: working on ros2_control

File: src/socks_bot/description/socks_bot.urdf (robot description, URDF)
Before this commit: robot sam_bot, 5 links, 4 joints
Links:
- removed link imu_link

Commit message: keep working

File: src/socks_bot/description/socks_bot.urdf (robot description, URDF)
Before this commit: robot sam_bot, 4 links, 4 joints
Joints:
- removed joint imu_joint
